File: Board Files/Motherboard.kicad_pcb (KiCad board)
At the start: 2 copper layers, 106.1 x 155 mm, 84 parts, among them P1 72-Pin Connector, P2 PowerSw, P3 ResetSw, P4 Controller_Port, P6 RF-Mod, Q1 2SA937, Q2 2SC2021, T1 08RB01, U1 6116 (WRAM), U2 74HC373, U3 74HC139, U4 6116 (VRAM), U5 RP2C02 PPU, U6 RP2A03 CPU, U7 40H368 (CI), U8 40H368 (CII), U9 L7805, X1 21.47727 MHz

Commit message: little bit of routing
Parts:
- removed  : TestPoint_Pad_D2.5mm, TestPoint:TestPoint_Pad_D2.5mm (x6)
- removed ACPLUG1: , Toploader:AC-JACK
- removed the C10 at (69.2, -110.8)
- removed DB1: RC203, Toploader:Rectifier
- removed P6: RF-Mod, Toploader:RF-MOD
- removed REF**: OSHW-Logo2_14.6x12mm_SilkScreen, Symbol:OSHW-Logo2_14.6x12mm_SilkScreen
- removed T1: 08RB01, Toploader:Inductor
- removed U9: L7805, Connector_PinHeader_2.54mm:PinHeader_1x03_P2.54mm_Vertical
- added C39: 1uF, Capacitor_THT:CP_Radial_D5.0mm_P2.50mm, F.Cu at (68.6, -11.9)
- added C8: 51pf, Capacitor_THT:C_Disc_D3.0mm_W2.0mm_P2.50mm, F.Cu at (170.5, -31.8)
- added J1: USB_C_Receptacle_PowerOnly_6P, Connector_USB:USB_C_Receptacle_GCT_USB4125-xx-x-0190_6P_TopMnt_Horizontal, F.Cu at (63.5, -2.54)
- added J2: Conn_Coaxial, Connector_Coaxial:BNC_Win_364A2x95_Horizontal, F.Cu at (159.0, -41.8)
- added J3: Left, Connector_Coaxial:BNC_Win_364A2x95_Horizontal, F.Cu at (176.1, -41.8)
- added J4: Right, Connector_Coaxial:BNC_Win_364A2x95_Horizontal, F.Cu at (193.1, -41.8)
- added Q3: AO3400A, Package_TO_SOT_SMD:SOT-23, F.Cu at (70.4, -16.6)
- added Q4: 2SC2021, Package_TO_SOT_THT:TO-126-3_Vertical, F.Cu at (224.5, -27.9)
- added Q5: BC817, Package_TO_SOT_SMD:SOT-23, F.Cu at (177.0, -25.2)
- added R11: 5.1K, Resistor_THT:R_Axial_DIN0207_L6.3mm_D2.5mm_P10.16mm_Horizontal, F.Cu at (61.7, -12.4)
- added R12: 5.1K, Resistor_THT:R_Axial_DIN0207_L6.3mm_D2.5mm_P10.16mm_Horizontal, F.Cu at (61.7, -8.64)
- added R13: 150K, Resistor_THT:R_Axial_DIN0207_L6.3mm_D2.5mm_P10.16mm_Horizontal, F.Cu at (203.2, -60.0)
- added R14: 560, Resistor_THT:R_Axial_DIN0207_L6.3mm_D2.5mm_P10.16mm_Horizontal, F.Cu at (203.2, -56.0)
- added R15: 75, Resistor_THT:R_Axial_DIN0207_L6.3mm_D2.5mm_P10.16mm_Horizontal, F.Cu at (203.2, -51.9)
- added R16: 330, Resistor_THT:R_Axial_DIN0207_L6.3mm_D2.5mm_P10.16mm_Horizontal, F.Cu at (222.5, -34.5)
- added U10: IP2721, Package_SO:TSSOP-16_4.4x5mm_P0.65mm, F.Cu at (63.5, -17.4)
- C10: renamed from C8; value 10nF -> 15pf
- C12: value 10nF -> 10uF; footprint Capacitor_THT:C_Disc_D3.0mm_W1.6mm_P2.50mm -> Capacitor_THT:CP_Radial_D5.0mm_P2.50mm
- C13: value 1500uF -> 51pf; footprint Capacitor_THT:CP_Radial_D12.5mm_P5.00mm -> Capacitor_THT:C_Disc_D3.0mm_W2.0mm_P2.50mm
- C14: value 1uF -> 10uf
- C18, C24: footprint Capacitor_THT:C_Disc_D3.0mm_W1.6mm_P2.50mm -> Capacitor_THT:C_Disc_D5.0mm_W2.5mm_P5.00mm
- C27, C30, C31, C36, C37, C38, C5, C6: footprint Capacitor_THT:C_Disc_D3.0mm_W2.0mm_P2.50mm -> Capacitor_THT:C_Disc_D5.0mm_W2.5mm_P5.00mm
- C28: footprint Capacitor_THT:C_Disc_D3.0mm_W2.0mm_P2.50mm -> Capacitor_THT:C_Disc_D6.0mm_W2.5mm_P5.00mm
- C7: value 330pF -> 220pf; footprint Capacitor_THT:C_Disc_D3.0mm_W1.6mm_P2.50mm -> Capacitor_THT:C_Disc_D3.0mm_W2.0mm_P2.50mm
- C9: value 10pF -> 18pf
- P2: footprint Toploader:PowerSwitchV2 -> Toploader:PowerSwitch
- P3: footprint Toploader:ResetSwitchV2 -> Toploader:ResetSwitch
- R10: value 150 -> 220K
- R2: value 430 -> 5.6K
- R3: value 150 -> 330
- R8: value 150K -> 510
- U7: value 40H368 (CI) -> 74HC368/40H368 (CI)
- U8: value 40H368 (CII) -> 74HC368/40H368 (CII)
- moved R2 138.1 mm to (222.5, -38.1), turned to 0 degrees
- moved C7 124.9 mm to (170.5, -35.3), turned to 0 degrees
- moved R3 113.3 mm to (203.2, -72.2), turned to 0 degrees
- moved C13 84.2 mm to (170.5, -28.2)
- moved C14 79.5 mm to (162.6, -33.0), turned to 0 degrees
- moved C12 9.86 mm to (54.0, -17.3), turned to 180 degrees
Connections:
- net /CPU-R~W renamed /CPU-R~{W}
- net /PPU-~A13 renamed /PPU-~{A13}
- net /PPU-~CE renamed /PPU-~{CE}
- net /PPU-~RD renamed /PPU-~{RD}
- net /PPU-~WE renamed /PPU-~{WE}
- net /VRAM-~CE renamed /VRAM-~{CE}
- net /WRAM-~CE renamed /WRAM-~{CE}
- net /~IRQ renamed /~{IRQ}
- net /~NMI renamed /~{NMI}
- net /~OE1 renamed /~{OE1}
- net /~OE2 renamed /~{OE2}
- net /~ROMSEL renamed /~{ROMSEL}
- net /~RST renamed /~{RST}
- BC1 pad 1: /GND -> GND
- BC1 pad 2: /VCC -> VCC
- C1 pad 1: /VCC -> VCC
- C1 pad 2: /GND -> GND
- C10 pad 1: Net-(C8-Pad1) -> Net-(Q2-C)
- C10 pad 2: /GND -> GND
- C11 pad 2: /GND -> GND
- C12 pad 1: Net-(ACPLUG1-Pad2) -> Net-(Q3-S)
- C12 pad 2: Net-(ACPLUG1-Pad1) -> GND
- C13 pad 1: Net-(C13-Pad1) -> Net-(Q2-B)
- C13 pad 2: /GND -> GND
- C14 pad 1: /VCC -> Net-(C14-Pad1)
- C14 pad 2: /GND -> /VIDEO
- C15 pad 2: /GND -> GND
- C16 pad 2: /GND -> GND
- C17 pad 2: /GND -> GND
- C18 pad 1: /VCC -> VCC
- C18 pad 2: /GND -> GND
- C19 pad 2: /GND -> GND
- C2 pad 1: /GND -> GND
- C20 pad 2: /GND -> GND
- C21 pad 2: /GND -> GND
- C22 pad 2: /GND -> GND
- C23 pad 2: /GND -> GND
- C24 pad 1: /VCC -> VCC
- C24 pad 2: /GND -> GND
- C25 pad 2: /GND -> GND
- C26 pad 2: /GND -> GND
- C27 pad 1: /GND -> GND
- C27 pad 2: /VCC -> VCC
- C28 pad 1: /GND -> GND
- C28 pad 2: /VCC -> VCC
- C29 pad 1: /GND -> GND
- C29 pad 2: /VCC -> VCC
- C30 pad 1: /GND -> GND
- C30 pad 2: /VCC -> VCC
- C31 pad 1: /GND -> GND
- C31 pad 2: /VCC -> VCC
- C32 pad 1: /GND -> GND
- C32 pad 2: /VCC -> VCC
- C33 pad 1: /GND -> GND
- C33 pad 2: /VCC -> VCC
- C34 pad 1: /GND -> GND
- C34 pad 2: /VCC -> VCC
- C35 pad 1: /GND -> GND
- C35 pad 2: /VCC -> VCC
- C36 pad 1: /GND -> GND
- C36 pad 2: /VCC -> VCC
- C37 pad 1: /GND -> GND
- C37 pad 2: /VCC -> VCC
- C38 pad 1: /GND -> GND
- C38 pad 2: /VCC -> VCC
- C4 pad 1: /GND -> GND
- C5 pad 2: /GND -> GND
- C6 pad 1: /GND -> GND
- C6 pad 2: /VCC -> VCC
- C7 pad 1: /GND -> /SYSTEM-CLK
- C7 pad 2: Net-(C7-Pad2) -> /CPU-CLK
- C9 pad 1: Net-(C9-Pad1) -> Net-(Q2-B)
- C9 pad 2: Net-(C7-Pad2) -> Net-(C9-Pad2)
- DA1 pad 4: /VCC -> VCC
- DA1 pad 7: /GND -> GND
- DA2 pad 4: /GND -> GND
- DA2 pad 7: /VCC -> VCC
- DA3 pad 1: /GND -> GND
- DA3 pad 4: /VCC -> VCC
- DA4 pad 1: /VCC -> VCC
- DA4 pad 4: /GND -> GND
- FC2 pad 1: Net-(FC2-Pad1) -> Net-(Q1-E)
- P1 pad 1: /GND -> GND
- P1 pad 34: Net-(P1-Pad34) -> unconnected-(P1-CIC-TO-CART-Pad34)
- P1 pad 35: Net-(P1-Pad35) -> unconnected-(P1-CIC-TO-MB-Pad35)
- P1 pad 36: /VCC -> VCC
- P1 pad 70: /VCC -> VCC
- P1 pad 72: /GND -> GND
- P2 pad 1: Net-(C13-Pad1) -> Net-(Q3-S)
- P2 pad 2: Net-(P2-Pad2) -> VCC
- P2 pad 3: /GND -> GND
- P3 pad 2: /GND -> GND
- P4 pad 1-1: /GND -> GND
- P4 pad 1-2: /GND -> GND
- P4 pad 3: /GND -> (no net)
- P4 pad 4: /GND -> (no net)
- P4 pad 5: /GND -> (no net)
- P4 pad 5-1: /VCC -> VCC
- P4 pad 5-2: /VCC -> VCC
- Q1 pad 1: Net-(Q1-Pad1) -> Net-(Q1-E)
- Q1 pad 2: /GND -> GND
- Q2 pad 1: Net-(C8-Pad1) -> GND
- Q2 pad 2: Net-(C10-Pad2) -> Net-(Q2-C)
- Q2 pad 3: Net-(C7-Pad2) -> Net-(Q2-B)
- R1 pad 1: /VCC -> VCC
- R1 pad 2: Net-(Q1-Pad1) -> Net-(Q1-E)
- R10 pad 1: Net-(C8-Pad1) -> Net-(Q2-B)
- R10 pad 2: /GND -> Net-(Q2-C)
- R2 pad 1: Net-(FC2-Pad1) -> VCC
- R2 pad 2: Net-(Q1-Pad1) -> Net-(Q5-B)
- R3 pad 1: /GND -> Net-(Q5-B)
- R3 pad 2: Net-(FC2-Pad1) -> GND
- R4 pad 1: /GND -> GND
- R5 pad 1: /GND -> GND
- R8 pad 1: Net-(C10-Pad2) -> /SYSTEM-CLK
- R8 pad 2: Net-(C7-Pad2) -> GND
- R9 pad 1: Net-(C10-Pad2) -> Net-(Q2-C)
- R9 pad 2: /VCC -> VCC
- RA1 pad 1: /VCC -> VCC
- TC1 pad 1: Net-(C9-Pad1) -> Net-(Q2-B)
- TC1 pad 2: Net-(C7-Pad2) -> Net-(C9-Pad2)
- U1 pad 12: /GND -> GND
- U1 pad 20: /GND -> GND
- U1 pad 24: /VCC -> VCC
- U2 pad 1: /GND -> GND
- U2 pad 10: /GND -> GND
- U2 pad 20: /VCC -> VCC
- U3 pad 10: Net-(U3-Pad10) -> unconnected-(U3B-O2-Pad10)
- U3 pad 12: Net-(U3-Pad12) -> unconnected-(U3B-O0-Pad12)
- U3 pad 15: /GND -> GND
- U3 pad 16: /VCC -> VCC
- U3 pad 6: Net-(U3-Pad6) -> unconnected-(U3A-O2-Pad6)
- U3 pad 7: Net-(U3-Pad7) -> unconnected-(U3A-O3-Pad7)
- U3 pad 8: /GND -> GND
- U4 pad 12: /GND -> GND
- U4 pad 24: /VCC -> VCC
- U5 pad 14: /GND -> GND
- U5 pad 15: /GND -> GND
- U5 pad 16: /GND -> GND
- U5 pad 17: /GND -> GND
- U5 pad 18: /SYS-CLK -> /PPU-CLK
- U5 pad 20: /GND -> GND
- U5 pad 22: /VCC -> VCC
- U5 pad 40: /VCC -> VCC
- U6 pad 20: /GND -> GND
- U6 pad 29: /SYS-CLK -> /CPU-CLK
- U6 pad 30: /GND -> GND
- U6 pad 40: /VCC -> VCC
- U7 pad 10: /VCC -> VCC
- U7 pad 12: /VCC -> VCC
- U7 pad 14: /VCC -> VCC
- U7 pad 16: /VCC -> VCC
- U7 pad 8: /GND -> GND
- U8 pad 10: /GND -> GND
- U8 pad 13: Net-(U8-Pad13) -> unconnected-(U8-~{6Y}-Pad13)
- U8 pad 14: /GND -> GND
- U8 pad 15: /GND -> GND
- U8 pad 16: /VCC -> VCC
- U8 pad 8: /GND -> GND
- U8 pad 9: Net-(U8-Pad9) -> unconnected-(U8-~{4Y}-Pad9)
- X1 pad 1: Net-(C10-Pad2) -> Net-(C9-Pad2)
- X1 pad 2: Net-(C9-Pad1) -> Net-(Q2-C)
Routing:
- net /VCC: track 477.6 -> 0.00 mm, vias 36 -> 0
- net (no net): track 0.00 -> 413.5 mm, vias 0 -> 26
- net VCC: track 0.00 -> 394.4 mm, vias 0 -> 11
- net Net-(P2-Pad2): track 229.2 -> 0.00 mm
- net Net-(Q3-S): track 0.00 -> 228.0 mm, vias 0 -> 1
- net GND: track 0.00 -> 227.3 mm, vias 0 -> 70
- net /GND: track 216.1 -> 23.8 mm, vias 78 -> 0
- net Net-(C13-Pad1): track 191.2 -> 0.00 mm
- net Net-(FC2-Pad1): track 98.7 -> 0.00 mm, vias 1 -> 0
- net /SYS-CLK: track 64.0 -> 0.00 mm, vias 1 -> 0
- net Net-(ACPLUG1-Pad2): track 35.4 -> 0.00 mm, vias 3 -> 0
- net Net-(ACPLUG1-Pad1): track 35.1 -> 0.00 mm, vias 4 -> 0
- net Net-(Q3-D): track 0.00 -> 25.8 mm
- net Net-(DB1-Pad4): track 20.4 -> 0.00 mm
- net Net-(J1-CC1): track 0.00 -> 18.0 mm
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- added copper zone on B.Cu, net /CPU-CLK
- added copper zone on B.Cu, net GND
- added copper zone on F.Cu, net GND
- added copper zone on B.Cu, net Net-(C9-Pad2)
- added copper zone on B.Cu, net VCC
- added copper zone on F.Cu, net VCC
- removed copper zone on B.Cu, net /GND
- removed copper zone on F.Cu, net /GND
- removed copper zone on B.Cu, net /SYS-CLK
- removed copper zone on B.Cu, net /VCC
- removed copper zone on F.Cu, net /VCC
- removed copper zone on B.Cu, net Net-(C10-Pad2)
- removed copper zone on B.Cu, net Net-(C7-Pad2)
Other:
- outline, holes or cut-outs redrawn
- net class Default removed
- net class Thin removed
- board text removed: "+"

Commit message: Progress
Parts:
- C27: footprint Capacitor_THT:C_Disc_D5.0mm_W2.5mm_P5.00mm -> Capacitor_THT:C_Disc_D3.0mm_W2.0mm_P2.50mm
- J2: value Conn_Coaxial -> Composite; footprint Connector_Coaxial:BNC_Win_364A2x95_Horizontal -> Samacsys:PJRAN1X1U03AUX
- J3, J4: footprint Connector_Coaxial:BNC_Win_364A2x95_Horizontal -> Samacsys:PJRAN1X1U03AUX
- moved R2 201.6 mm to (22.1, -16.5)
- moved R16 185.2 mm to (37.5, -25.5), turned to 180 degrees
- moved R14 183.0 mm to (23.1, -23.5), turned to 180 degrees
- moved R15 182.9 mm to (23.1, -20.0), turned to 180 degrees
- moved R3 178.6 mm to (32.2, -20.5)
- moved J4 169.6 mm to (28.2, -2.31)
- moved Q4 169.2 mm to (81.8, -118.9)
- moved R13 153.9 mm to (62.7, -122.9)
- moved J2 150.5 mm to (13.8, -2.42)
- moved Q5 148.9 mm to (28.2, -20.3)
- moved J3 139.0 mm to (42.7, -2.42)
- moved C13 129.5 mm to (78.0, -118.9), turned to 180 degrees
- moved C7 127.0 mm to (71.9, -115.3), turned to 90 degrees
- moved C8 124.8 mm to (71.9, -108.3), turned to 90 degrees
- moved C14 120.8 mm to (42.0, -25.5)
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Routing:
- net (no net): track 413.5 -> 138.6 mm, vias 26 -> 21
- net Net-(Q1-E): track 11.1 -> 119.6 mm
- net /CPU-CLK: track 0.00 -> 48.2 mm
- net Net-(Q2-C): track 0.00 -> 36.8 mm
- net Net-(Q3-S): track 228.0 -> 193.9 mm
- net /PPU-D4: track 174.2 -> 142.0 mm, vias 4 -> 1
- net /PPU-D7: track 157.4 -> 125.8 mm, vias 3 -> 1
- net VCC: track 394.4 -> 363.8 mm, vias 11 -> 10
- net /PPU-D6: track 161.7 -> 133.4 mm, vias 3 -> 1
- net /PPU-D5: track 174.5 -> 148.2 mm, vias 3 -> 1
- net /AUDIO: track 88.2 -> 114.4 mm
- net /GND: track 23.8 -> 0.00 mm
- net Net-(Q2-B): track 0.00 -> 21.2 mm
- net Net-(J2-In): track 0.00 -> 17.7 mm
- net Net-(Q1-B): track 48.4 -> 32.8 mm
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
Commit message: all connected up
Parts:
- removed C13: 51pf, Capacitor_THT:C_Disc_D3.0mm_W2.0mm_P2.50mm
- removed the C8 at (71.9, -108.3)
- removed Q4: 2SC2021, Package_TO_SOT_THT:TO-126-3_Vertical
- removed the R8 at (87.1, -126.2)
- added C10: 330pf, Capacitor_THT:C_Disc_D3.0mm_W1.6mm_P2.50mm, F.Cu at (68.5, -111.0)
- C18, C24, C30, C31, C36, C37, C38: footprint Capacitor_THT:C_Disc_D5.0mm_W2.5mm_P5.00mm -> Capacitor_THT:C_Disc_D3.0mm_W1.6mm_P2.50mm
- C28: footprint Capacitor_THT:C_Disc_D6.0mm_W2.5mm_P5.00mm -> Capacitor_THT:C_Disc_D3.0mm_W1.6mm_P2.50mm
- C7: renamed from C10; value 15pf -> 330pf; footprint Capacitor_THT:C_Disc_D3.0mm_W2.0mm_P2.50mm -> Capacitor_THT:C_Disc_D3.0mm_W1.6mm_P2.50mm
- C8: renamed from C7; value 220pf -> 10nf
- C9: value 18pf -> 10pf
- R10: value 220K -> 150
- moved R8 21.8 mm to (79.2, -108.8)
- moved C11 21.3 mm to (90.0, -134.3), turned to -90 degrees
- moved C7 17.4 mm to (76.2, -118.2), turned to 90 degrees
- moved C8 16.6 mm to (81.8, -102.0), turned to 180 degrees
- moved C9 8.30 mm to (86.7, -118.2), turned to 90 degrees
- moved R10 5.55 mm to (72.0, -118.6), turned to -90 degrees
- moved TC1 4.94 mm to (81.8, -118.5), turned to 90 degrees
- moved C38 3.85 mm to (68.5, -115.9)
- moved X1 3.78 mm to (86.7, -113.5)
- moved C35 2.62 mm to (68.4, -94.4), turned to 90 degrees
- moved C37 1.20 mm to (43.2, -114.7)
- moved R9 0.62 mm to (79.2, -105.2)
- moved Q2 0.33 mm to (76.2, -108.5)
- moved C30 0.14 mm to (51.6, -59.4)
- moved C28 0.10 mm to (51.6, -48.2)
- renumbered R13 to R8
Connections:
- C7 pad 1: Net-(Q2-C) -> Net-(Q2-B)
- C8 pad 1: /SYSTEM-CLK -> GND
- C8 pad 2: /CPU-CLK -> Net-(Q2-E)
- C9 pad 1: Net-(Q2-B) -> Net-(C9-Pad1)
- C9 pad 2: Net-(C9-Pad2) -> Net-(Q2-B)
- P1 pad 37: /SYSTEM-CLK -> /SYS-CLK
- Q2 pad 1: GND -> Net-(Q2-E)
- R10 pad 1: Net-(Q2-B) -> GND
- R10 pad 2: Net-(Q2-C) -> Net-(Q2-E)
- R8 pad 1: /CPU-CLK -> Net-(Q2-C)
- R8 pad 2: GND -> Net-(Q2-B)
- TC1 pad 1: Net-(Q2-B) -> Net-(C9-Pad1)
- TC1 pad 2: Net-(C9-Pad2) -> Net-(Q2-B)
- U5 pad 18: /PPU-CLK -> /SYS-CLK
- U6 pad 29: /CPU-CLK -> /SYS-CLK
- X1 pad 1: Net-(C9-Pad2) -> Net-(Q2-C)
- X1 pad 2: Net-(Q2-C) -> Net-(C9-Pad1)
Routing:
- net VCC: track 363.8 -> 591.4 mm, vias 10 -> 9
- net /SYS-CLK: track 0.00 -> 165.5 mm, vias 0 -> 1
- net (no net): track 138.6 -> 0.00 mm, vias 21 -> 0
- net /CPU-CLK: track 48.2 -> 0.00 mm
- net Net-(C9-Pad2): track 14.8 -> 0.00 mm
- net Net-(Q2-E): track 0.00 -> 12.0 mm
- net Net-(Q2-B): track 21.2 -> 32.4 mm
- net Net-(Q2-C): track 36.8 -> 26.0 mm
- net Net-(C9-Pad1): track 0.00 -> 10.0 mm
- net /SYSTEM-CLK: track 9.57 -> 0.00 mm
- net /~{RST}: track 141.0 -> 131.6 mm
- net /PPU-CLK: track 6.28 -> 0.00 mm
- net GND: track 232.2 -> 234.6 mm, vias 66 -> 46
- net Net-(Q3-S): track 193.9 -> 191.9 mm
- net Net-(Q5-E): track 9.98 -> 7.94 mm
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- removed copper zone on B.Cu, net /CPU-CLK
- removed copper zone on B.Cu, net Net-(C9-Pad2)
- removed copper zone on B.Cu, net VCC

Commit message: 4 Layer complete
Parts:
- C12, C39: footprint Capacitor_THT:CP_Radial_D5.0mm_P2.50mm -> Capacitor_THT:CP_Radial_D6.3mm_P2.50mm
- moved C12 22.3 mm to (75.7, -11.4)
- moved R1 16.5 mm to (89.4, -101.1), turned to -90 degrees
- moved C5 10.6 mm to (37.1, -17.3), turned to 0 degrees
- moved U10 8.91 mm to (72.2, -19.1), turned to -90 degrees
- moved C39 8.38 mm to (64.3, -19.1), turned to 0 degrees
- moved R11 8.18 mm to (69.8, -13.3)
- moved R12 8.18 mm to (69.8, -9.53)
- moved J1 7.15 mm to (70.6, -3.34)
- moved Q3 7.05 mm to (77.0, -19.1)
- moved Q1 6.06 mm to (85.9, -90.9)
- moved FC1 2.83 mm to (10.7, -59.5)
- moved C36 0.39 mm to (14.2, -118.1)
- moved DA1 0.33 mm to (34.9, -128.3)
- moved R3 0.30 mm to (32.0, -20.3)
- moved DA3 0.29 mm to (14.6, -128.3)
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Routing:
- net VCC: track 591.4 -> 40.2 mm, vias 9 -> 1
- net GND: track 234.6 -> 26.7 mm, vias 46 -> 40
- net Net-(Q3-S): track 191.9 -> 141.6 mm, vias 1 -> 0
- net Net-(Q3-D): track 25.8 -> 42.7 mm
- net /4016-D4: track 85.7 -> 100.5 mm
- net /PPU-D5: track 148.2 -> 136.9 mm
- net /AUDIO: track 114.4 -> 105.0 mm, vias 1 -> 0
- net /PPU-D1: track 148.3 -> 139.1 mm, vias 3 -> 1
- net /PPU-D2: track 141.0 -> 132.4 mm, vias 3 -> 2
- net Net-(Q1-E): track 119.6 -> 112.6 mm
- net /PPU-A7: track 37.9 -> 31.3 mm
- net /PPU-D3: track 131.1 -> 125.7 mm, vias 5 -> 3
- net /M2: track 101.9 -> 97.0 mm, vias 2 -> 1
- net /~{OE1}: track 77.3 -> 82.0 mm
- net /4016-D0: track 58.1 -> 62.0 mm
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- added copper zone on In1.Cu, net GND
- added copper zone on In2.Cu, net VCC
- removed copper zone on F.Cu, net GND
- removed copper zone on F.Cu, net VCC
Other:
- copper layers 2 -> 4
