File: Board Files/Motherboard.kicad_sch (KiCad schematic)
At the start: 84 parts, among them J1 USB_C_Receptacle_PowerOnly_6P, J2 Composite, J3 Left, J4 Right, P1 72-Pin Connector, P2 PowerSw, P3 ResetSw, P4 Controller_Port, Q1 2SA937, Q2 2SC2021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

Commit message: 4 Layer complete
Parts:
- C12, C39: footprint Capacitor_THT:CP_Radial_D5.0mm_P2.50mm -> Capacitor_THT:CP_Radial_D6.3mm_P2.50mm
Changed lines of the file:
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@@
 			)
 		)
-		(property "Footprint" "Capacitor_THT:CP_Radial_D5.0mm_P2.50mm"
+		(property "Footprint" "Capacitor_THT:CP_Radial_D6.3mm_P2.50mm"
 			(at 374.65 176.53 0)
 			(effects
@@
 			)
 		)
-		(property "Footprint" "Capacitor_THT:CP_Radial_D5.0mm_P2.50mm"
+		(property "Footprint" "Capacitor_THT:CP_Radial_D6.3mm_P2.50mm"
 			(at 331.47 158.75 0)
 			(effects
